Commit message: Add files via upload

File: urdf/robot.xacro (robot description, xacro)
@@ -116,5 +116,5 @@
     <axis xyz="0 0 0" />
    <!-- <origin xyz="${camera_link} 0 ${height3 - axel_offset*2}" rpy="0 0 0"/> -->
-    <origin xyz = "0 ${0.07+camera_link/2} 0" rpy = "0 0.78539 1.5708"/>
+    <origin xyz = "0 ${0.07+camera_link/2} 0" rpy = "0 0.52359877559 1.5708"/>
     <parent link="chassis"/>
     <child link="camera_link"/>
@@ -163,10 +163,10 @@
                channels, which at that point lie in the range [0,1]. -->
           <mean>0.0</mean>
-          <stddev>0.007</stddev>
+          <stddev>0.00</stddev>
         </noise>
       </camera>
       <plugin name="camera_controller" filename="libgazebo_ros_camera.so">
         <alwaysOn>true</alwaysOn>
-        <updateRate>0.01</updateRate>
+        <updateRate>100</updateRate>
         <cameraName>rrbot/camera1</cameraName>
         <imageTopicName>image_raw</imageTopicName>
